File: pcb/pcb.sch (KiCad schematic (older format))
At the start: 62 parts, among them J1 TYPE-C-31-M-12, J2 AudioJack4, J3 AudioJack4, SW1 SW_Push, SW10 SW_Push, SW11 SW_Push, SW12 SW_Push, SW13 SW_Push, SW14 SW_Push, SW15 SW_Push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

Commit message: parts align (without trrs jack)
Parts:
- C1, C2, C3, C4, R1, R2, R3, R4, R5: footprint (none) -> SMD:2012M
- D1, D10, D11, D12, D13, D14, D15, D16, D17, D18, D19, D2, D20, D21, D22, D23, D24, D3, D4, D5, D6, D7, D8, D9: footprint (none) -> SMD:SOD123
- J1: footprint USB_Type-C:HRO_TYPE-C-31-M-12 -> USB_Type-C:TYPE-C-31-M-12
- SW1, SW10, SW11, SW12, SW13, SW14, SW15, SW16, SW17, SW18, SW19, SW2, SW20, SW21, SW22, SW23, SW24, SW3, SW4, SW5, SW6, SW7, SW8, SW9: footprint Cherry_MX:1u_socket -> Cherry_MX:1u

Commit message: routing done
Parts:
- J2, J3: footprint (none) -> Phone_Connector:MJ-4PP-9
Connections:
- net C0: now also U1.31 (PC6); no longer U1.8 (PB0)
- net C1: now also U1.30 (PB6); no longer U1.9 (PB1)
- net C2: now also U1.29 (PB5); no longer U1.10 (PB2)
- net C3: now also U1.36 (PF7); no longer U1.11 (PB3)
- net C4: now also U1.39 (PF4); no longer U1.28 (PB4)
- net C5: now also U1.38 (PF5); no longer U1.29 (PB5)
- net R1: now also U1.28 (PB4); no longer U1.40 (PF1)
- net R2: now also U1.27 (PD7); no longer U1.39 (PF4)
- net R3: now also U1.26 (PD6); no longer U1.38 (PF5)
- net SCL: now also J2.R2, J3.R2; no longer J2.R1, J3.R1
- net SDA: now also J2.R1, J3.R1; no longer J2.R2, J3.R2
- no-connect marks 16 -> 12
Changed lines of the file:
@@
 F 0 "J2" H 8757 6025 50  0000 C CNN
 F 1 "AudioJack4" H 8757 5934 50  0000 C CNN
-F 2 "" H 8800 5700 50  0001 C CNN
+F 2 "Phone_Connector:MJ-4PP-9" H 8800 5700 50  0001 C CNN
 F 3 "~" H 8800 5700 50  0001 C CNN
 	1    8800 5700
@@
 	0    -1   -1   0
 $EndComp
+Text GLabel 9000 5800 2    50   Input ~ 0
+SDA
 Text GLabel 9000 5700 2    50   Input ~ 0
-SDA
-Text GLabel 9000 5800 2    50   Input ~ 0
 SCL
 $Comp
@@
 Text GLabel 5300 1300 1    50   Input ~ 0
 C5
-Text GLabel 9600 1500 2    50   Input ~ 0
+Text GLabel 9600 2400 2    50   Input ~ 0
 C0
-Text GLabel 9600 1600 2    50   Input ~ 0
+Text GLabel 9600 2100 2    50   Input ~ 0
 C1
-Text GLabel 9600 1700 2    50   Input ~ 0
+Text GLabel 9600 2000 2    50   Input ~ 0
 C2
-Text GLabel 9600 1800 2    50   Input ~ 0
+Text GLabel 9600 4400 2    50   Input ~ 0
 C3
-Text GLabel 9600 1900 2    50   Input ~ 0
+Text GLabel 9600 4100 2    50   Input ~ 0
 C4
-Text GLabel 9600 2000 2    50   Input ~ 0
+Text GLabel 9600 4200 2    50   Input ~ 0
 C5
 Text GLabel 9600 3900 2    50   Input ~ 0
 R0
-Text GLabel 9600 4000 2    50   Input ~ 0
+Text GLabel 9600 1900 2    50   Input ~ 0
 R1
-Text GLabel 9600 4100 2    50   Input ~ 0
+Text GLabel 9600 3400 2    50   Input ~ 0
 R2
-Text GLabel 9600 4200 2    50   Input ~ 0
+Text GLabel 9600 3300 2    50   Input ~ 0
 R3
 $Comp
@@
 Wire Wire Line
 	7000 1500 7000 1600
-NoConn ~ 9600 2100
 NoConn ~ 9600 2200
 NoConn ~ 9600 2900
@@
 NoConn ~ 9600 3100
 NoConn ~ 9600 3200
-NoConn ~ 9600 3300
-NoConn ~ 9600 3400
 NoConn ~ 9600 3700
-NoConn ~ 9600 4300
-NoConn ~ 9600 4400
 $Comp
 L power:VCC #PWR05
@@
 Text GLabel 7700 4550 2    50   Input ~ 0
 D-
-NoConn ~ 9600 2400
 NoConn ~ 9600 2500
 $Comp
@@
 F 0 "J3" H 9757 6025 50  0000 C CNN
 F 1 "AudioJack4" H 9757 5934 50  0000 C CNN
-F 2 "" H 9800 5700 50  0001 C CNN
+F 2 "Phone_Connector:MJ-4PP-9" H 9800 5700 50  0001 C CNN
 F 3 "~" H 9800 5700 50  0001 C CNN
 	1    9800 5700
@@
 	0    -1   -1   0
 $EndComp
+Text GLabel 10000 5800 2    50   Input ~ 0
+SDA
 Text GLabel 10000 5700 2    50   Input ~ 0
-SDA
-Text GLabel 10000 5800 2    50   Input ~ 0
 SCL
 $Comp
@@
 Wire Wire Line
 	6500 2600 6500 2700
+NoConn ~ 9600 4300
+NoConn ~ 9600 4000
 $EndSCHEMATC

Commit message: + reset button
Parts:
- added R6: 10k, SMD:2012M, symbol Device:R
- added RST1: SW_Push, Button_Switch_SMD:SW_SPST_TL3342, symbol Switch:SW_Push
Connections:
- net GND: now also RST1.1
- net RESET: now also R6.1, RST1.2
- net VCC: now also R6.2
Changed lines of the file:
@@
 NoConn ~ 9600 4300
 NoConn ~ 9600 4000
+Text GLabel 7500 3250 2    50   Input ~ 0
+RESET
+$Comp
+L Device:R R6
+U 1 1 5F3A3460
+P 7100 3050
+F 0 "R6" V 7000 3050 50  0000 C CNN
+F 1 "10k" V 7100 3050 50  0000 C CNN
+F 2 "SMD:2012M" V 7030 3050 50  0001 C CNN
+F 3 "~" H 7100 3050 50  0001 C CNN
+	1    7100 3050
+	0    1    1    0
+$EndComp
+$Comp
+L power:VCC #PWR0101
+U 1 1 5F3A44BF
+P 6800 2950
+F 0 "#PWR0101" H 6800 2800 50  0001 C CNN
+F 1 "VCC" H 6817 3123 50  0000 C CNN
+F 2 "" H 6800 2950 50  0001 C CNN
+F 3 "" H 6800 2950 50  0001 C CNN
+	1    6800 2950
+	1    0    0    -1
+$EndComp
+Wire Wire Line
+	6800 2950 6800 3050
+Wire Wire Line
+	7400 3250 7500 3250
+$Comp
+L Switch:SW_Push RST1
+U 1 1 5F3B82D1
+P 7100 3250
+F 0 "RST1" H 7100 3150 50  0000 C CNN
+F 1 "SW_Push" H 7100 3444 50  0001 C CNN
+F 2 "Button_Switch_SMD:SW_SPST_TL3342" H 7100 3450 50  0001 C CNN
+F 3 "~" H 7100 3450 50  0001 C CNN
+	1    7100 3250
+	1    0    0    -1
+$EndComp
+Wire Wire Line
+	7400 3050 7400 3250
+Wire Wire Line
+	7300 3250 7400 3250
+Connection ~ 7400 3250
+$Comp
+L power:GND #PWR0102
+U 1 1 5F3D8444
+P 6800 3350
+F 0 "#PWR0102" H 6800 3100 50  0001 C CNN
+F 1 "GND" H 6805 3177 50  0000 C CNN
+F 2 "" H 6800 3350 50  0001 C CNN
+F 3 "" H 6800 3350 50  0001 C CNN
+	1    6800 3350
+	1    0    0    -1
+$EndComp
+Wire Wire Line
+	6800 3350 6800 3250
+Wire Wire Line
+	6800 3250 6900 3250
+Wire Wire Line
+	7250 3050 7400 3050
+Wire Wire Line
+	6800 3050 6950 3050
 $EndSCHEMATC
