File: pcb/pcb.kicad_pcb (KiCad board)
At the start: 2 copper layers, 115.2 x 76.8 mm, 64 parts, among them J1 TYPE-C-31-M-12, J2 AudioJack4, J3 AudioJack4, SW1 SW_Push, SW10 SW_Push, SW11 SW_Push, SW12 SW_Push, SW13 SW_Push, SW14 SW_Push, SW15 SW_Push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

Commit message: + I2C pullup
Parts:
- added R7: 5.1k, SMD:2012M, B.Cu at (85.2, 34.8)
- added R8: 5.1k, SMD:2012M, B.Cu at (85.2, 36.8)
Routing:
- net VCC: track 207.5 -> 222.9 mm, vias 4 -> 6
- net SDA: track 141.8 -> 148.3 mm
- net SCL: track 146.8 -> 153.0 mm
Other:
- board text added: "I2C"
